File: bombay_beats_button_module.kicad_sch (KiCad schematic)
At the start: 2 parts, among them SW1 SW_Push_Dual

Commit message: fix 0603 footprints
Parts:
- R1: footprint Resistor_SMD:R_0201_0603Metric -> Resistor_SMD:R_0603_1608Metric; LCSC Part #  C328335 -> C25804
Changed lines of the file:
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@@
 			)
 		)
-		(property "Footprint" "Resistor_SMD:R_0201_0603Metric"
+		(property "Footprint" "Resistor_SMD:R_0603_1608Metric"
 			(at 72.644 42.164 90)
 			(effects
@@
 			)
 		)
-		(property "LCSC Part # " "C328335"
+		(property "LCSC Part # " "C25804"
 			(at 72.39 43.18 90)
 			(effects
